Commit message: Add lidar plugin to vehicle
Lidar is not completely set up yet but the plugin exists on the robot

File: ackermann_vehicle/ackermann_vehicle_description/urdf/em_3905.urdf.xacro (robot description, xacro)
@@ -97,4 +97,5 @@
   <!-- Camera -->
   <xacro:property name="camera_link" value="0.05" /> <!-- Size of square 'camera' box -->
+  <xacro:property name="lidar_size" value="0.05" /> <!-- Size of square 'camera' box -->
   <material name="battery_mat">
     <color rgba="0 0 1 1"/>
@@ -348,17 +349,20 @@
     <child link="chassis"/>
   </joint>
-  <!-- Camera Joint -->
-  <joint name="camera_joint" type="fixed">
+  <!-- ##### -->
+  <!-- Lidar -->
+  <!-- ##### -->
+  <!-- Lidar Joint -->
+  <joint name="lidar_joint" type="fixed">
     <axis xyz="0 1 0" />
-    <origin xyz="${camera_link + 0.4} 0 ${chassis_height + 0.5}" rpy="0 1.21 0" />
+    <origin xyz="${lidar_size + 0.4} 0 ${chassis_height + 0.5}" rpy="0 1.21 0" />
     <parent link="chassis" />
-    <child link="camera_link" />
+    <child link="lidar_link" />
   </joint>
-  <!-- Camera -->
-  <link name="camera_link">
+  <!-- Lidar Link -->
+  <link name="lidar_link">
     <collision>
       <origin xyz="0 0 0" rpy="0 0 0"/>
       <geometry>
-    <box size="${camera_link} ${camera_link} ${camera_link}"/>
+    <box size="${lidar_size} ${lidar_size} ${lidar_size}"/>
       </geometry>
     </collision>
@@ -366,5 +370,5 @@
       <origin xyz="0 0 0" rpy="0 0 0"/>
       <geometry>
-    <box size="${camera_link} ${camera_link} ${camera_link}"/>
+    <box size="${lidar_size} ${lidar_size} ${lidar_size}"/>
       </geometry>
       <material name="red"/>
@@ -376,5 +380,71 @@
     </inertial>
   </link>
-  <!-- camera -->
+  <gazebo reference="hokuyo_link">
+    <sensor type="ray" name="laser_sensor">
+      <pose>0 0 0 0 0 0</pose>
+      <visualize>false</visualize>
+      <update_rate>30</update_rate>
+      <ray>
+        <scan>
+          <horizontal>
+            <samples>180</samples>
+            <resolution>1</resolution>
+            <min_angle>-1.570796</min_angle>
+            <max_angle>1.570796</max_angle>
+          </horizontal>
+        </scan>
+        <range>
+          <min>0.10</min>
+          <max>30.0</max>
+          <resolution>0.01</resolution>
+        </range>
+        <noise>
+          <type>gaussian</type>
+          <!-- Noise parameters based on published spec for Hokuyo laser
+               achieving "+-30mm" accuracy at range < 10m.  A mean of 0.0m and
+               stddev of 0.01m will put 99.7% of samples within 0.03m of the true
+               reading. -->
+          <mean>0.0</mean>
+          <stddev>0.01</stddev>
+        </noise>
+      </ray>
+      <plugin name="gazebo_ros_laser_controller" filename="libgazebo_ros_laser.so">
+        <topicName>/lidar2d/scan</topicName>
+        <frameName>lidar_link</frameName>
+      </plugin>
+    </sensor>
+  </gazebo>
+  <!-- ###### -->
+  <!-- Camera -->
+  <!-- ###### -->
+  <!-- Camera Joint -->
+  <joint name="camera_joint" type="fixed">
+    <axis xyz="0 1 0" />
+    <origin xyz="${camera_link + 0.4} 0 ${chassis_height + 0.5}" rpy="0 1.21 0" />
+    <parent link="chassis" />
+    <child link="camera_link" />
+  </joint>
+  <!-- Camera Link -->
+  <link name="camera_link">
+    <collision>
+      <origin xyz="0 0 0" rpy="0 0 0"/>
+      <geometry>
+    <box size="${camera_link} ${camera_link} ${camera_link}"/>
+      </geometry>
+    </collision>
+    <visual>
+      <origin xyz="0 0 0" rpy="0 0 0"/>
+      <geometry>
+    <box size="${camera_link} ${camera_link} ${camera_link}"/>
+      </geometry>
+      <material name="red"/>
+    </visual>
+    <inertial>
+      <mass value="1e-5" />
+      <origin xyz="0 0 0" rpy="0 0 0"/>
+      <inertia ixx="1e-6" ixy="0" ixz="0" iyy="1e-6" iyz="0" izz="1e-6" />
+    </inertial>
+  </link>
+  <!-- Camera -->
   <gazebo reference="camera_link">
     <sensor type="camera" name="camera1">

Commit message: Adjust lidar parameters, attach to correct link

File: ackermann_vehicle/ackermann_vehicle_description/urdf/em_3905.urdf.xacro (robot description, xacro)
@@ -355,5 +355,5 @@
   <joint name="lidar_joint" type="fixed">
     <axis xyz="0 1 0" />
-    <origin xyz="${lidar_size + 0.4} 0 ${chassis_height + 0.5}" rpy="0 1.21 0" />
+    <origin xyz="0.1 0 ${chassis_height + 0.1}" rpy="0 0 0" />
     <parent link="chassis" />
     <child link="lidar_link" />
@@ -380,8 +380,8 @@
     </inertial>
   </link>
-  <gazebo reference="hokuyo_link">
-    <sensor type="ray" name="laser_sensor">
+  <gazebo reference="lidar_link">
+    <sensor type="ray" name="head_hokuyo_sensor">
       <pose>0 0 0 0 0 0</pose>
-      <visualize>false</visualize>
+      <visualize>true</visualize>
       <update_rate>30</update_rate>
       <ray>
@@ -396,5 +396,5 @@
         <range>
           <min>0.10</min>
-          <max>30.0</max>
+          <max>5.0</max>
           <resolution>0.01</resolution>
         </range>
@@ -409,5 +409,5 @@
         </noise>
       </ray>
-      <plugin name="gazebo_ros_laser_controller" filename="libgazebo_ros_laser.so">
+      <plugin name="gazebo_ros_head_hokuyo_controller" filename="libgazebo_ros_laser.so">
         <topicName>/lidar2d/scan</topicName>
         <frameName>lidar_link</frameName>
